File: PingPong1975.kicad_sch (KiCad schematic)
At the start: 77 parts, among them SW1 Reset, U1 28C256, U10 74100, U11 74100, U12 74100, U2 74LS04, U3 8205/74LS138, U4 74HC4051, U5 74LS02, U6 AM93L422PC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

Commit message: Primeras versiones pintando en el osciloscopio
Parts:
- ROM: renamed from U1; value 28C256 -> 28C64
Connections:
- net DAC1_RD renamed DAC1_WR
- net DAC2_RD renamed DAC2_WR
Changed lines of the file:
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@@
 	)
 	(bus_entry
-		(at 208.28 63.5)
-		(size 2.54 2.54)
-		(stroke
-			(width 0)
-			(type default)
-		)
-	)
-	(bus_entry
 		(at 236.22 135.89)
 		(size 2.54 2.54)
@@
 	)
 	(bus_entry
-		(at 208.28 60.96)
-		(size 2.54 2.54)
-		(stroke
-			(width 0)
-			(type default)
-		)
-	)
-	(bus_entry
 		(at 238.76 107.95)
 		(size 2.54 2.54)
@@
 		)
 	)
-	(bus
-		(pts
-			(xy 208.28 60.96) (xy 208.28 63.5)
-		)
-		(stroke
-			(width 0)
-			(type default)
-		)
-	)
 	(wire
 		(pts
@@
 	(bus
 		(pts
-			(xy 208.28 58.42) (xy 208.28 60.96)
-		)
-		(stroke
-			(width 0)
-			(type default)
-		)
-	)
-	(bus
-		(pts
 			(xy 115.57 161.29) (xy 115.57 175.26)
 		)
@@
 	(wire
 		(pts
-			(xy 210.82 66.04) (xy 212.09 66.04)
-		)
-		(stroke
-			(width 0)
-			(type default)
-		)
-	)
-	(wire
-		(pts
 			(xy 186.69 361.95) (xy 186.69 364.49)
 		)
@@
 	(wire
 		(pts
-			(xy 210.82 63.5) (xy 212.09 63.5)
-		)
-		(stroke
-			(width 0)
-			(type default)
-		)
-	)
-	(wire
-		(pts
 			(xy 118.11 236.22) (xy 120.65 236.22)
 		)
@@
 		)
 	)
-	(text_box "Dreccionamiento:\n\nROM: 0x0000-0x1FFF (A13=0)\nRAM: 0x2000-0xFFFF (A13=1)"
+	(text_box "Direccionamiento:\n\nROM: 0x0000-0x1FFF (A13=0) (8 kilobytes)\nRAM: 0x2000-0x20FF (A13=1) (256 bytes)"
 		(exclude_from_sim no)
-		(at 134.62 45.72 0)
-		(size 35.56 10.16)
+		(at 234.95 76.2 0)
+		(size 46.99 10.16)
 		(stroke
 			(width 0)
@@
 		)
 	)
-	(text_box "No es necesaria la OR del esquema original ya que la EEPROM 28C256 tiene dos entradas para activarla (CE y OE) mientras que la PROM 8207 solo tenia una (CS/WE)"
+	(text_box "No es necesaria la OR del esquema original ya que la EEPROM 28C64 tiene dos entradas para activarla (CE y OE) mientras que la PROM 8207 solo tenia una (CS/WE)"
 		(exclude_from_sim no)
 		(at 236.22 55.88 0)
@@
 		)
 	)
-	(label "DAC2_RD"
+	(label "DAC2_WR"
 		(at 92.71 210.82 0)
 		(fields_autoplaced yes)
@@
 		)
 	)
-	(label "DAC1_RD"
+	(label "DAC1_WR"
 		(at 92.71 200.66 0)
 		(fields_autoplaced yes)
@@
 		(dnp no)
 		(fields_autoplaced yes)
-		(property "Reference" "U1"
+		(property "Reference" "ROM"
 			(at 224.4441 22.86 0)
 			(effects
@@
 			)
 		)
-		(property "Value" "28C256"
+		(property "Value" "28C64"
 			(at 224.4441 25.4 0)
 			(effects
@@
 			)
 		)
-		(pin "1"
-		)
 		(pin "7"
 		)
@@
 		(pin "20"
 		)
-		(pin "26"
-		)
 		(instances
 			(project ""
 				(path "/925f831f-14fc-49d2-bb8a-562ceac93277"
-					(reference "U1")
+					(reference "ROM")
 					(unit 1)
 				)

Commit message: Prototipo funcionando al 100% con codigo sin modificar
Parts:
- removed R50, R51: 10K, symbol Device:R
- removed U8: 74LS08, symbol 74xx:74LS08
- added U1: 74LS32, symbol 74xx:74LS32
- added U13, U8: 74LS126, symbol 74xx:74LS126
- added U2: 74LS04, symbol 74xx:74LS04
- added unit 1 of U2
- added unit 5 of U2
Connections:
- net ADC_RD: now also U13.1, U13.10, U13.13, U13.4, U8.1, U8.10, U8.13, U8.4
- net D0: now also U8.3; no longer ADC.18 (DB0)
- net D1: now also U8.6; no longer ADC.17 (DB1)
- net D2: now also U8.8; no longer ADC.16 (DB2)
- net D3: now also U8.11; no longer ADC.15 (DB3)
- net D4: now also U13.3; no longer ADC.14 (DB4)
- net D5: now also U1.1, U13.6; no longer ADC.13 (DB5)
- net D6: now also U13.8; no longer ADC.12 (DB6)
- net D7: now also U13.11; no longer ADC.11 (DB7)
- net GND: now also ADC.1 (~{CS})
- net at U11.5 (1Q1): now also U2.1; no longer R52.1
- net at U2.4: now also U1.2
- net at ADC.3 (~{WR}): now also U1.3
- net at U10.5 (1Q1): now also U2.3; no longer R27.1
- new net: U13.12, U2.10
- new net: ADC.12 (DB6), U13.9
- new net: R27.1, U2.4
- new net: R52.1, U2.2
- new net: ADC.17 (DB1), U8.5
- new net: ADC.11 (DB7), U2.11
- new net: ADC.13 (DB5), U13.5
- new net: ADC.18 (DB0), U8.2
- new net: ADC.14 (DB4), U13.2
- new net: ADC.15 (DB3), U8.12
- new net: ADC.16 (DB2), U8.9
Other:
- moved on the sheet: U10
